File: board/power.kicad_sch (KiCad schematic)
At the start: 10 parts, among them U2 AP63203WU-7

Commit message: Schematic and Layout Complete
Parts:
- added D5: D_TVS, Diode_SMD:D_SMA, symbol Device:D_TVS
- added D6: D_Schottky, Diode_SMD:D_SOD-123F, symbol Device:D_Schottky
- added F1: 2A, Fuse:Fuse_1206_3216Metric_Pad1.42x1.75mm_HandSolder, symbol Device:Fuse
- L1: footprint SignalStack:INDM2520X190N -> Inductor_SMD:L_1812_4532Metric_Pad1.30x3.40mm_HandSolder
Connections:
- net GND: now also D5.1 (A1)
- net VIN: now also F1.1; no longer C1.1, D2.2 (A), U2.2 (EN), U2.3 (VIN)
- new net: C1.1, D2.2 (A), D5.2 (A2), D6.1 (K), U2.2 (EN), U2.3 (VIN)
- new net: D6.2 (A), F1.2
